File: KiCad/BBC Hat.sch (KiCad schematic (older format))
At the start: 6 parts, among them P11 CONN_20X2

Commit message: Routine
Parts:
- added P? (x3): CONN_02X06, symbol CONN_02X06
Connections:
- net labels added: 14_V, CAN1_H, CAN1_L, CAN2_H, CAN2_L

Commit message: Routine
Parts:
- added C? (x2): 220uF, symbol CP
- added C? (x2): 100nF, symbol C
- added D?: DIODE_SCHOTTKY, Pkg, symbol DIODE_SCHOTTKY
- added L?: INDUCTOR, symbol INDUCTOR
- added U?: AP1509, symbol AP1509
Connections:
- net labels added: 5v, ANV0, ANV1, ANV10, ANV11, ANV12, ANV13, ANV14, ANV15, ANV2, ANV3, ANV4, ANV5, ANV6, ANV7, ANV8, ANV9, GPIO1, GPIO2, GPIO3, GPIO4, GPIO5, SLI1_MISO, SLI1_MOSI, SPI1_CLK, TIMER1, TIMER2, TIMER3, TIMER4
- wire segments 13 -> 22
Other:
- moved on the sheet: P11, P?
