File: KiCad/STM32.sch (KiCad schematic (older format))
At the start: 14 parts, among them P1 CONN_01X05, SW1 Boot, U1 STM32F107VCTx, U2 SN65HVD233, U3 SN65HVD233

Commit message: Routine
Parts:
- R1: value R -> 10k
Connections:
- net PULL_10: now reaches U1.1 (PE2/SYS_TRACECLK)
- net PULL_11: now reaches U1.2 (PE3/SYS_TRACED0)
- net PULL_12: now reaches U1.3 (PE4/SYS_TRACED1)
- net PULL_15: now reaches U1.38 (PE7/TIM1_ETR)
- net PULL_13: now reaches U1.4 (PE5/SYS_TRACED2)
- net TIM1_CH3: now reaches U1.44 (PE13/TIM1_CH3)
- net TIM2_CH3: now reaches U1.47 (ETH_RX_ER/TIM2_CH3/USART3_TX/PB10)
- net PULL_14: now reaches U1.5 (PE6/SYS_TRACED3)
- net TIM3_CH3: now reaches U1.65 (TIM3_CH3/PC8)
- net PC10: now reaches U1.78 (I2S3_CK/SPI3_SCK/UART4_TX/USART3_TX/PC10)
- net PC11: now reaches U1.79 (ADC1_EXTI11/ADC2_EXTI11/SPI3_MISO/UART4_RX/USART3_RX/PC11)
- net PC12: now reaches U1.80 (I2S3_SD/SPI3_MOSI/UART5_TX/USART3_CK/PC12)
- net PULL_GPIO1: now reaches U1.81 (PD0/CAN1_RX)
- net PULL_GPIO2: now reaches U1.82 (PD1/CAN1_TX)
- net PULL_GPIO3: now reaches U1.83 (PD2/TIM3_ETR/UART5_RX)
- net PULL_GPIO4: now reaches U1.84 (PD3/USART2_CTS)
- net PULL_GPIO5: now reaches U1.85 (PD4/USART2_RTS)
- net SPI1_CLK: now reaches U1.89 (I2S3_CK/SPI1_SCK/SPI3_SCK/SYS_JTDO/SYS_TRACESWO/TIM2_CH2/PB3)
- net SPI1_MISO: now reaches U1.90 (SPI1_MISO/SPI3_MISO/SYS_NJTRST/TIM3_CH1/PB4)
- net SPI1_MOSI: now reaches U1.91 (CAN2_RX/ETH_PPS_OUT/I2C1_SMBA/I2S3_SD/SPI1_MOSI/SPI3_MOSI/TIM3_CH2/PB5)
- net TIM4_CH1: now reaches U1.92 (CAN2_TX/I2C1_SCL/TIM4_CH1/USART1_TX/PB6)
- net PB8: now reaches U1.95 (CAN1_RX/ETH_TXD3/I2C1_SCL/TIM4_CH3/PB8)
- net PB9: now reaches U1.96 (CAN1_TX/DAC_EXTI9/I2C1_SDA/TIM4_CH4/PB9)
Changed lines of the file:
@@
 P 1600 3000
 F 0 "R1" H 1670 3046 50  0000 L CNN
-F 1 "R" H 1670 2955 50  0000 L CNN
+F 1 "10k" H 1670 2955 50  0000 L CNN
 F 2 "" V 1530 3000 50  0000 C CNN
 F 3 "" H 1600 3000 50  0000 C CNN
@@
 Wire Wire Line
 	8650 5550 7650 5550
+Text GLabel 2250 4550 0    60   Input ~ 0
+PULL_10
+Text GLabel 2250 4650 0    60   Input ~ 0
+PULL_11
+Text GLabel 2250 4750 0    60   Input ~ 0
+PULL_12
+Text GLabel 2250 4850 0    60   Input ~ 0
+PULL_13
+Text GLabel 2250 4950 0    60   Input ~ 0
+PULL_14
+Text GLabel 2250 5050 0    60   Input ~ 0
+PULL_15
+Text GLabel 7650 4650 2    60   Input ~ 0
+SPI1_CLK
+Text GLabel 7650 4750 2    60   Input ~ 0
+SPI1_MISO
+Text GLabel 7650 4850 2    60   Input ~ 0
+SPI1_MOSI
+Text GLabel 2250 5650 0    60   Input ~ 0
+TIM1_CH3
+Text GLabel 7650 5350 2    60   Input ~ 0
+TIM2_CH3
+Text GLabel 7650 6850 2    60   Input ~ 0
+TIM3_CH3
+Text GLabel 7650 4950 2    60   Input ~ 0
+TIM4_CH1
+Text GLabel 2250 6050 0    60   Input ~ 0
+PULL_GPIO1
+Text GLabel 2250 6150 0    60   Input ~ 0
+PULL_GPIO2
+Text GLabel 2250 6250 0    60   Input ~ 0
+PULL_GPIO3
+Text GLabel 2250 6350 0    60   Input ~ 0
+PULL_GPIO4
+Text GLabel 2250 6450 0    60   Input ~ 0
+PULL_GPIO5
+Text GLabel 7650 7050 2    60   Input ~ 0
+PC10
+Text GLabel 7650 7150 2    60   Input ~ 0
+PC11
+Text GLabel 7650 7250 2    60   Input ~ 0
+PC12
+Text GLabel 7650 5250 2    60   Input ~ 0
+PB9
+Text GLabel 7650 5150 2    60   Input ~ 0
+PB8
 $EndSCHEMATC
