File: KiCad/Sensors.sch (KiCad schematic (older format))
At the start: 2 parts

Commit message: Routine
Parts:
- removed Q?: MOSFET_P_DEPLETION, Pkg, symbol MOSFET_P_DEPLETION
Changed lines of the file:
@@
 	1    0    0    -1
 $EndComp
-$Comp
-L MOSFET_P_DEPLETION Q?
-U 0 1 58E75495
-P 7650 2200
-F 0 "Q?" H 7791 2117 60  0000 L CNN
-F 1 "MOSFET_P_DEPLETION" H 7791 2223 60  0000 L CNN
-F 2 "Pkg" H 7791 2306 30  0000 L CNN
-F 3 "" H 7650 2200 60  0000 C CNN
-	0    7650 2200
-	1    0    0    1
-$EndComp
 $EndSCHEMATC
